File: IR2_Projetos de PCB/ir2_B2_UFAM/Módulo AmplInst.kicad_sch (KiCad schematic)
At the start: 23 parts, among them J8 Entrada, J9 Saída, U6 LMC7660, U7 AD620, U8 ir2_U8_LM358

Commit message: Alterado 3D da placa.
Parts:
- U8: footprint SOP100P600X150-8N -> IR2_Library:IR2_UFAM_V1_LM358
Changed lines of the file:
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@@
 			)
 		)
-		(property "Footprint" "SOP100P600X150-8N"
+		(property "Footprint" "IR2_Library:IR2_UFAM_V1_LM358"
 			(at 98.12 74.93 0)
 			(effects
