File: IR2_Projetos de PCB/ir2_B2_UFAM/ir2_B2_UFAM.kicad_pcb (KiCad board)
At the start: 2 copper layers, 100 x 100 mm, 67 parts, among them IC1 LM358, J1 NC3MBH-B, J2 USBAsp, J3 IR2_UFAM_V0_PLCC84, J4 DE15_Socket_HighDensity_Mount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, J5 Conn_01x03_Pin, J6 Conn_01x03_Pin, J7 Conn_01x03_Pin, J8 Entrada, J9 Saída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

Commit message: commit 2
Digitação e atualização teste
Other:
- board text added: "Projeto IR2 B2 UFAM 2026 V1 24/08/2025"
- board text removed: "Projeto IR2 B2 UFAM 2026 V0"
Changed lines of the file:
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@@
 		)
 	)
-	(gr_text "Projeto IR2 B2 UFAM 2026 V0"
+	(gr_text "Projeto IR2 B2 UFAM 2026 V1\n24/08/2025"
 		(at 182.04 133.66 0)
 		(layer "F.SilkS")

Commit message: Alterado 3D da placa.
Parts:
- renumbered IC1 to U8
Changed lines of the file:
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@@
 		(embedded_fonts no)
 		(model "${KICAD9_3DMODEL_DIR}/LIB_PLCC-84-AT/PLCC-84-AT/3D/PLCC-84-AT.stp"
+			(hide yes)
 			(offset
 				(xyz 0 -15.23999954 -0.05999999776)
@@
 			)
 		)
-		(model "${KICAD9_3DMODEL_DIR}/ir2_J3_PLCC-84-AT.3dshapes/ir2_J3_PLCC-84-AT.stp"
+		(model "G:/Kicad/share/kicad/3dmodels/ir2_J3_PLCC-84-AT.3dshapes/ir2_J3_PLCC-84-AT.stp"
 			(offset
 				(xyz 0 -15.5 0)
@@
 		(embedded_fonts no)
 		(model "${KICAD9_3DMODEL_DIR}/LED_THT.3dshapes/LED_D5.0mm.step"
+			(hide yes)
+			(offset
+				(xyz 0 0 0)
+			)
+			(scale
+				(xyz 1 1 1)
+			)
+			(rotate
+				(xyz 0 0 0)
+			)
+		)
+		(model "${KICAD9_3DMODEL_DIR}/LED_THT.3dshapes/LED_D3.0mm_Green.step"
+			(offset
+				(xyz 0 0 0)
+			)
+			(scale
+				(xyz 1 1 1)
+			)
+			(rotate
+				(xyz 0 0 0)
+			)
+		)
+		(model "${KICAD9_3DMODEL_DIR}/LED_THT.3dshapes/LED_D5.0mm_Green.step"
 			(offset
 				(xyz 0 0 0)
@@
 		(embedded_fonts no)
 		(model "${KICAD9_3DMODEL_DIR}/Connector_Audio.3dshapes/Jack_XLR_Neutrik_NC3MBH-B_Horizontal.step"
+			(hide yes)
 			(offset
 				(xyz 0 0 0)
@@
 			)
 		)
-		(model "${KICAD9_3DMODEL_DIR}/LIB_NC3MBH-B.3dshapes/ir2_J1_NC3MBH-B.stp"
+		(model "${KIPRJMOD}/IR2_Library.pretty/IR2_UFAM_V0_NC3MBH-B.kicad_sym"
+			(hide yes)
+			(offset
+				(xyz 0 0 0)
+			)
+			(scale
+				(xyz 1 1 1)
+			)
+			(rotate
+				(xyz -0 -0 180)
+			)
+		)
+		(model "${KICAD9_3DMODEL_DIR}/NC3MBH-B.3dshapes/NC3MBH-B.stp"
 			(offset
 				(xyz 0 0 0)
@@
 		(embedded_fonts no)
 		(model "${KICAD9_3DMODEL_DIR}/LED_THT.3dshapes/LED_D5.0mm.step"
+			(hide yes)
+			(offset
+				(xyz 0 0 0)
+			)
+			(scale
+				(xyz 1 1 1)
+			)
+			(rotate
+				(xyz 0 0 0)
+			)
+		)
+		(model "${KICAD9_3DMODEL_DIR}/LED_THT.3dshapes/LED_D3.0mm_Blue.step"
+			(offset
+				(xyz 0 0 0)
+			)
+			(scale
+				(xyz 1 1 1)
+			)
+			(rotate
+				(xyz 0 0 0)
+			)
+		)
+		(model "${KICAD9_3DMODEL_DIR}/LED_THT.3dshapes/LED_D3.0mm_Green.step"
+			(offset
+				(xyz 0 0 0)
+			)
+			(scale
+				(xyz 1 1 1)
+			)
+			(rotate
+				(xyz 0 0 0)
+			)
+		)
+		(model "${KICAD9_3DMODEL_DIR}/LED_THT.3dshapes/LED_D5.0mm_Blue.step"
+			(offset
+				(xyz 0 0 0)
+			)
+			(scale
+				(xyz 1 1 1)
+			)
+			(rotate
+				(xyz 0 0 0)
+			)
+		)
+		(model "${KICAD9_3DMODEL_DIR}/LED_THT.3dshapes/LED_D5.0mm_Blue.step"
 			(offset
 				(xyz 0 0 0)
@@
 		(descr "SOIC, 8 Pin (JEITA/EIAJ ED-7311-19 variation 08-001-BBA and Atmel/Microchip, 208 mils width, https://www.jeita.or.jp/japanese/standard/book/ED-7311-19/#target/page_no=21, https://ww1.microchip.com/downloads/en/DeviceDoc/20005045C.pdf#page=23, https://ww1.microchip.com/downloads/en/DeviceDoc/doc2535.pdf#page=162), generated with kicad-footprint-generator ipc_gullwing_generator.py")
 		(tags "SOIC SO P-SOP SOP SOP-8 SO SO-8 8S2 S2AE/F K04-056 CASE-751BE SO8W 8-Pin-SOIC PSA W8-2 W8-4 W8MS-1 FPT-8P-M08")
-		(property "Reference" "IC1"
+		(property "Reference" "U8"
 			(at 0 -3.6 0)
 			(unlocked yes)
 			(layer "F.SilkS")
-			(hide yes)
 			(effects
 				(font
